Commit message: Commit before data collection on labor pc

File: simulation/firmware_files/urdf/iris_vl53l1x_lidars.urdf (robot description, URDF)
Before this commit: robot iris_vl53l1x_lidars, 4 links, 3 joints
Joints:
- joint laser_top_joint: origin xyz=0 0 0.1 rpy=0 0 0 -> xyz=0 0 0.06 rpy=0 0 0
