Commit message: Save progress

File: simulation/catkin_ws/install_isolated/share/cartographer_ros/urdf/iris_vl53l1x_lidars.urdf (robot description, URDF)
Before this commit: robot iris_vl53l1x_lidars, 4 links, 3 joints
Links:
- removed link laser_bottom
- removed link laser_top
- added link laser_bottom_link; visual box size=0.01 0.01 0.01
- added link laser_top_link; visual box size=0.01 0.01 0.01
Joints:
- joint imu_link_joint: origin xyz=0 0 0 rpy=0 -0 0 -> xyz=0 0 0 rpy=0 0 0
- joint laser_bottom_joint: child laser_bottom -> laser_bottom_link
- joint laser_top_joint: child laser_top -> laser_top_link; origin xyz=0 0 0.1 rpy=0 0 0 -> xyz=0 0 0.06 rpy=0 0 0
